Commit message: use configurable wheel collision width

File: src/scrobot_description/urdf/wheels.xacro (robot description, xacro)
@@ -24,5 +24,5 @@
         <origin xyz="0 0 0" rpy="${pi/2} 0 0"/>
         <geometry>
-          <cylinder radius="${wheel_radius}" length="${wheel_width}"/>
+          <cylinder radius="${wheel_radius}" length="${wheel_collision_width}"/>
         </geometry>
       </collision>
