Commit message: Simplify collector frame and add physical collision

File: src/scrobot_description/urdf/collector.xacro (robot description, xacro)
@@ -3,15 +3,4 @@
   <xacro:macro name="scrobot_collector">
     <link name="collector_link">
-      <inertial>
-        <origin xyz="0 -0.0023 0" rpy="0 0 0"/>
-        <mass value="0.150"/>
-        <inertia
-          ixx="1.24e-3"
-          ixy="0"
-          ixz="0"
-          iyy="6.41e-5"
-          iyz="0"
-          izz="1.24e-3"/>
-      </inertial>
       <visual name="collector_visual">
         <origin xyz="0 0 0" rpy="0 0 0"/>
@@ -21,4 +10,11 @@
         <material name="plastic_blue"/>
       </visual>
+      <!-- Simple physical roller collision; detailed STL remains visual-only. -->
+      <collision name="collector_collision">
+        <origin xyz="0 0 0" rpy="${pi/2} 0 0"/>
+        <geometry>
+          <cylinder radius="${collector_radius}" length="${collector_length}"/>
+        </geometry>
+      </collision>
     </link>
     <joint name="collector_joint" type="fixed">
@@ -27,10 +23,4 @@
       <origin xyz="${collector_x} ${collector_y} ${collector_z}" rpy="0 0 0"/>
     </joint>
-    <link name="pickup_link"/>
-    <joint name="pickup_joint" type="fixed">
-      <parent link="collector_link"/>
-      <child link="pickup_link"/>
-      <origin xyz="0 0 0" rpy="0 0 0"/>
-    </joint>
   </xacro:macro>
 </robot>

Commit message: Remove floor-contacting fixed collector collision

File: src/scrobot_description/urdf/collector.xacro (robot description, xacro)
@@ -3,4 +3,19 @@
   <xacro:macro name="scrobot_collector">
     <link name="collector_link">
+      <!--
+        Keep collector_link as a real Gazebo/TF link with negligible placeholder
+        inertia. The assembled-body mass/inertia remains owned by base_link.
+      -->
+      <inertial>
+        <origin xyz="0 0 0" rpy="0 0 0"/>
+        <mass value="0.0001"/>
+        <inertia
+          ixx="1e-8"
+          ixy="0"
+          ixz="0"
+          iyy="1e-8"
+          iyz="0"
+          izz="1e-8"/>
+      </inertial>
       <visual name="collector_visual">
         <origin xyz="0 0 0" rpy="0 0 0"/>
@@ -10,11 +25,12 @@
         <material name="plastic_blue"/>
       </visual>
-      <!-- Simple physical roller collision; detailed STL remains visual-only. -->
-      <collision name="collector_collision">
-        <origin xyz="0 0 0" rpy="${pi/2} 0 0"/>
-        <geometry>
-          <cylinder radius="${collector_radius}" length="${collector_length}"/>
-        </geometry>
-      </collision>
+      <!--
+        Intentionally no collision geometry here. At the current mount height
+        the physical 60 mm roller touches the court. Modelling it as a fixed
+        cylinder makes Gazebo treat the collector as a non-rotating floor skid
+        and can prevent the drive wheels from moving the chassis. Shuttle
+        pickup physics uses collector_link pose + pickup envelope in the
+        simulation plugin instead.
+      -->
     </link>
     <joint name="collector_joint" type="fixed">
