Commit message: add control thru cmd_vel_manual/approach/nav

File: src/scrobot_description/urdf/base.xacro (robot description, xacro)
@@ -3,8 +3,21 @@
   <xacro:macro name="scrobot_base">
     <!--
-      base_footprint is the planar navigation reference on the floor.
-      base_link is the physical chassis reference at the chassis centre.
+      Planar navigation reference.
+      This is primarily a TF frame, but because it is the root link of
+      the URDF we give it a very small non-zero inertia for Gazebo.
     -->
-    <link name="base_footprint"/>
+    <link name="base_footprint">
+      <inertial>
+        <origin xyz="0 0 0" rpy="0 0 0"/>
+        <mass value="0.001"/>
+        <inertia
+          ixx="0.000001"
+          ixy="0.0"
+          ixz="0.0"
+          iyy="0.000001"
+          iyz="0.0"
+          izz="0.000001"/>
+      </inertial>
+    </link>
     <joint name="base_footprint_joint" type="fixed">
       <parent link="base_footprint"/>
@@ -12,4 +25,5 @@
       <origin xyz="0 0 ${base_link_z}" rpy="0 0 0"/>
     </joint>
+    <!-- Physical chassis -->
     <link name="base_link">
       <visual>
@@ -26,4 +40,17 @@
         </geometry>
       </collision>
+      <inertial>
+        <origin xyz="0 0 0" rpy="0 0 0"/>
+        <!-- Placeholder mass -->
+        <mass value="10.0"/>
+        <!-- Inertia of a rectangular box -->
+        <inertia
+          ixx="${10.0 / 12.0 * (base_width * base_width + base_height * base_height)}"
+          ixy="0.0"
+          ixz="0.0"
+          iyy="${10.0 / 12.0 * (base_length * base_length + base_height * base_height)}"
+          iyz="0.0"
+          izz="${10.0 / 12.0 * (base_length * base_length + base_width * base_width)}"/>
+      </inertial>
     </link>
   </xacro:macro>

File: src/scrobot_description/urdf/collector.xacro (robot description, xacro)
@@ -15,4 +15,15 @@
         </geometry>
       </collision>
+      <inertial>
+        <origin xyz="0 0 0" rpy="0 0 0"/>
+        <mass value="1.0"/>
+        <inertia
+          ixx="${1.0 / 12.0 * (collector_width * collector_width + collector_height * collector_height)}"
+          ixy="0.0"
+          ixz="0.0"
+          iyy="${1.0 / 12.0 * (collector_length * collector_length + collector_height * collector_height)}"
+          iyz="0.0"
+          izz="${1.0 / 12.0 * (collector_length * collector_length + collector_width * collector_width)}"/>
+      </inertial>
     </link>
     <joint name="collector_joint" type="fixed">

File: src/scrobot_description/urdf/sensors.xacro (robot description, xacro)
@@ -10,4 +10,15 @@
         <material name="scrobot_sensor"/>
       </visual>
+      <inertial>
+        <origin xyz="0 0 0" rpy="0 0 0"/>
+        <mass value="0.2"/>
+        <inertia
+          ixx="0.00021"
+          ixy="0.0"
+          ixz="0.0"
+          iyy="0.00010"
+          iyz="0.0"
+          izz="0.00023"/>
+      </inertial>
     </link>
     <joint name="camera_joint" type="fixed">
@@ -43,4 +54,15 @@
         <material name="scrobot_sensor"/>
       </visual>
+      <inertial>
+        <origin xyz="0 0 0" rpy="0 0 0"/>
+        <mass value="0.05"/>
+        <inertia
+          ixx="0.0000076"
+          ixy="0.0"
+          ixz="0.0"
+          iyy="0.0000076"
+          iyz="0.0"
+          izz="0.0000133"/>
+      </inertial>
     </link>
     <joint name="imu_joint" type="fixed">

File: src/scrobot_description/urdf/wheels.xacro (robot description, xacro)
@@ -17,4 +17,15 @@
         </geometry>
       </collision>
+      <inertial>
+        <origin xyz="0 0 0" rpy="0 0 0"/>
+        <mass value="0.5"/>
+        <inertia
+          ixx="${0.5 / 12.0 * (3.0 * wheel_radius * wheel_radius + wheel_width * wheel_width)}"
+          ixy="0.0"
+          ixz="0.0"
+          iyy="${0.5 / 2.0 * wheel_radius * wheel_radius}"
+          iyz="0.0"
+          izz="${0.5 / 12.0 * (3.0 * wheel_radius * wheel_radius + wheel_width * wheel_width)}"/>
+      </inertial>
     </link>
     <joint name="${name}_wheel_joint" type="continuous">
