Commit message: add model, mass, inertia and collision

File: src/scrobot_description/urdf/base.xacro (robot description, xacro)
@@ -2,20 +2,9 @@
 <robot xmlns:xacro="http://www.ros.org/wiki/xacro">
   <xacro:macro name="scrobot_base">
-    <!--
-      Planar navigation reference.
-      This is primarily a TF frame, but because it is the root link of
-      the URDF we give it a very small non-zero inertia for Gazebo.
-    -->
     <link name="base_footprint">
       <inertial>
         <origin xyz="0 0 0" rpy="0 0 0"/>
-        <mass value="0.001"/>
-        <inertia
-          ixx="0.000001"
-          ixy="0.0"
-          ixz="0.0"
-          iyy="0.000001"
-          iyz="0.0"
-          izz="0.000001"/>
+        <mass value="0.0001"/>
+        <inertia ixx="1e-8" ixy="0" ixz="0" iyy="1e-8" iyz="0" izz="1e-8"/>
       </inertial>
     </link>
@@ -23,34 +12,31 @@
       <parent link="base_footprint"/>
       <child link="base_link"/>
-      <origin xyz="0 0 ${base_link_z}" rpy="0 0 0"/>
+      <origin xyz="0 0 ${wheel_radius}" rpy="0 0 0"/>
     </joint>
-    <!-- Physical chassis -->
     <link name="base_link">
-      <visual>
+      <inertial>
+        <origin xyz="-0.060 0.002 0.195" rpy="0 0 0"/>
+        <mass value="14.14"/>
+        <inertia
+          ixx="0.766"
+          ixy="0.00107"
+          ixz="0.338"
+          iyy="1.060"
+          iyz="-0.00308"
+          izz="0.727"/>
+      </inertial>
+      <visual name="base_visual">
         <origin xyz="0 0 0" rpy="0 0 0"/>
         <geometry>
-          <box size="${base_length} ${base_width} ${base_height}"/>
+          <mesh filename="package://scrobot_description/meshes/visual/base.STL" scale="1 1 1"/>
         </geometry>
-        <material name="scrobot_gray"/>
+        <material name="aluminum_grey"/>
       </visual>
-      <collision>
+      <collision name="base_collision">
         <origin xyz="0 0 0" rpy="0 0 0"/>
         <geometry>
-          <box size="${base_length} ${base_width} ${base_height}"/>
+          <mesh filename="package://scrobot_description/meshes/collision/base_collision.STL" scale="1 1 1"/>
         </geometry>
       </collision>
-      <inertial>
-        <origin xyz="0 0 0" rpy="0 0 0"/>
-        <!-- Placeholder mass -->
-        <mass value="10.0"/>
-        <!-- Inertia of a rectangular box -->
-        <inertia
-          ixx="${10.0 / 12.0 * (base_width * base_width + base_height * base_height)}"
-          ixy="0.0"
-          ixz="0.0"
-          iyy="${10.0 / 12.0 * (base_length * base_length + base_height * base_height)}"
-          iyz="0.0"
-          izz="${10.0 / 12.0 * (base_length * base_length + base_width * base_width)}"/>
-      </inertial>
     </link>
   </xacro:macro>

File: src/scrobot_description/urdf/collector.xacro (robot description, xacro)
@@ -2,46 +2,34 @@
 <robot xmlns:xacro="http://www.ros.org/wiki/xacro">
   <xacro:macro name="scrobot_collector">
-    <!-- Physical collector assembly. -->
     <link name="collector_link">
-      <visual>
+      <inertial>
+        <origin xyz="0 -0.0023 0" rpy="0 0 0"/>
+        <mass value="0.150"/>
+        <inertia
+          ixx="1.24e-3"
+          ixy="0"
+          ixz="0"
+          iyy="6.41e-5"
+          iyz="0"
+          izz="1.24e-3"/>
+      </inertial>
+      <visual name="collector_visual">
+        <origin xyz="0 0 0" rpy="0 0 0"/>
         <geometry>
-          <box size="${collector_length} ${collector_width} ${collector_height}"/>
+          <mesh filename="package://scrobot_description/meshes/visual/collector.STL" scale="1 1 1"/>
         </geometry>
-        <material name="scrobot_collector"/>
+        <material name="plastic_blue"/>
       </visual>
-      <collision>
-        <geometry>
-          <box size="${collector_length} ${collector_width} ${collector_height}"/>
-        </geometry>
-      </collision>
-      <inertial>
-        <origin xyz="0 0 0" rpy="0 0 0"/>
-        <mass value="1.0"/>
-        <inertia
-          ixx="${1.0 / 12.0 * (collector_width * collector_width + collector_height * collector_height)}"
-          ixy="0.0"
-          ixz="0.0"
-          iyy="${1.0 / 12.0 * (collector_length * collector_length + collector_height * collector_height)}"
-          iyz="0.0"
-          izz="${1.0 / 12.0 * (collector_length * collector_length + collector_width * collector_width)}"/>
-      </inertial>
     </link>
     <joint name="collector_joint" type="fixed">
       <parent link="base_link"/>
       <child link="collector_link"/>
-      <!-- Put the collector directly in front of the chassis and close to the floor. -->
-      <origin
-        xyz="${base_length / 2.0 + collector_length / 2.0} 0 ${collector_height / 2.0 - base_link_z}"
-        rpy="0 0 0"/>
+      <origin xyz="${collector_x} ${collector_y} ${collector_z}" rpy="0 0 0"/>
     </joint>
-    <!--
-      Functional operating point used later for shuttle approach/alignment.
-      It is located at the front-centre edge of the collector on the floor.
-    -->
     <link name="pickup_link"/>
     <joint name="pickup_joint" type="fixed">
       <parent link="collector_link"/>
       <child link="pickup_link"/>
-      <origin xyz="${collector_length / 2.0} 0 ${-collector_height / 2.0}" rpy="0 0 0"/>
+      <origin xyz="0 0 0" rpy="0 0 0"/>
     </joint>
   </xacro:macro>

File: src/scrobot_description/urdf/scrobot.urdf.xacro (robot description, xacro)
@@ -1,40 +1,60 @@
 <?xml version="1.0"?>
 <robot xmlns:xacro="http://www.ros.org/wiki/xacro" name="scrobot">
-  <!--
-    Placeholder dimensions for the first TF/URDF bring-up.
-    Replace these values with measured CAD dimensions later.
-    SI units: metres, kilograms, radians.
-  -->
-  <xacro:property name="base_length" value="0.60"/>
-  <xacro:property name="base_width" value="0.45"/>
-  <xacro:property name="base_height" value="0.15"/>
-  <xacro:property name="ground_clearance" value="0.05"/>
-  <xacro:property name="base_link_z" value="${ground_clearance + base_height / 2.0}"/>
-  <xacro:property name="wheel_radius" value="0.08"/>
-  <xacro:property name="wheel_width" value="0.04"/>
-  <xacro:property name="wheel_separation" value="0.49"/>
-  <xacro:property name="wheel_x" value="0.0"/>
-  <xacro:property name="collector_length" value="0.25"/>
-  <xacro:property name="collector_width" value="0.35"/>
-  <xacro:property name="collector_height" value="0.04"/>
-  <material name="scrobot_gray">
-    <color rgba="0.55 0.55 0.55 1.0"/>
+  <material name="aluminum_grey">
+    <color rgba="0.60 0.62 0.65 1.0"/>
   </material>
-  <material name="scrobot_dark">
-    <color rgba="0.12 0.12 0.12 1.0"/>
+  <material name="rubber_black">
+    <color rgba="0.03 0.03 0.03 1.0"/>
   </material>
-  <material name="scrobot_sensor">
-    <color rgba="0.20 0.35 0.80 1.0"/>
+  <material name="plastic_blue">
+    <color rgba="0.05 0.25 0.80 1.0"/>
   </material>
-  <material name="scrobot_collector">
-    <color rgba="0.85 0.55 0.10 1.0"/>
+  <material name="sensor_blue">
+    <color rgba="0.05 0.15 0.90 1.0"/>
   </material>
+  <xacro:property name="wheel_radius" value="0.050"/>
+  <xacro:property name="wheel_width" value="0.030"/>
+  <xacro:property name="wheel_separation" value="0.420"/>
+  <xacro:property name="base_front_x" value="0.325"/>
+  <xacro:property name="base_rear_x" value="-0.450"/>
+  <xacro:property name="base_left_y" value="0.225"/>
+  <xacro:property name="base_right_y" value="-0.225"/>
+  <xacro:property name="caster_x" value="-0.300"/>
+  <xacro:property name="caster_y" value="0.160"/>
+  <xacro:property name="caster_z" value="0.0085"/>
+  <xacro:property name="caster_radius" value="0.020"/>
+  <xacro:property name="caster_width" value="0.020"/>
+  <xacro:property name="caster_trail" value="-0.020"/>
+  <xacro:property name="caster_axle_drop" value="0.0385"/>
+  <xacro:property name="caster_fork_com_x" value="-0.00525"/>
+  <xacro:property name="caster_fork_com_y" value="0.0"/>
+  <xacro:property name="caster_fork_com_z" value="-0.01513"/>
+  <xacro:property name="collector_radius" value="0.030"/>
+  <xacro:property name="collector_diameter" value="0.060"/>
+  <xacro:property name="collector_length" value="0.300"/>
+  <xacro:property name="collector_x" value="0.165"/>
+  <xacro:property name="collector_y" value="0.0"/>
+  <xacro:property name="collector_z" value="-0.020"/>
+  <xacro:property name="camera_x" value="0.130"/>
+  <xacro:property name="camera_y" value="0.0"/>
+  <xacro:property name="camera_z" value="0.225"/>
+  <xacro:property name="camera_roll" value="0.0"/>
+  <xacro:property name="camera_pitch" value="${7.0 * pi / 180.0}"/>
+  <xacro:property name="camera_yaw" value="0.0"/>
+  <xacro:property name="imu_x" value="-0.035"/>
+  <xacro:property name="imu_y" value="0.0"/>
+  <xacro:property name="imu_z" value="0.030"/>
+  <xacro:property name="mag_x" value="-0.035"/>
+  <xacro:property name="mag_y" value="0.0"/>
+  <xacro:property name="mag_z" value="0.040"/>
   <xacro:include filename="$(find scrobot_description)/urdf/base.xacro"/>
   <xacro:include filename="$(find scrobot_description)/urdf/wheels.xacro"/>
+  <xacro:include filename="$(find scrobot_description)/urdf/casters.xacro"/>
+  <xacro:include filename="$(find scrobot_description)/urdf/collector.xacro"/>
   <xacro:include filename="$(find scrobot_description)/urdf/sensors.xacro"/>
-  <xacro:include filename="$(find scrobot_description)/urdf/collector.xacro"/>
   <xacro:scrobot_base/>
   <xacro:scrobot_wheels/>
+  <xacro:scrobot_casters/>
+  <xacro:scrobot_collector/>
   <xacro:scrobot_sensors/>
-  <xacro:scrobot_collector/>
 </robot>

File: src/scrobot_description/urdf/sensors.xacro (robot description, xacro)
@@ -1,73 +1,94 @@
 <?xml version="1.0"?>
 <robot xmlns:xacro="http://www.ros.org/wiki/xacro">
+  <xacro:macro name="tiny_sensor_inertial">
+    <inertial>
+      <origin xyz="0 0 0" rpy="0 0 0"/>
+      <mass value="0.0001"/>
+      <inertia ixx="1e-8" ixy="0" ixz="0" iyy="1e-8" iyz="0" izz="1e-8"/>
+    </inertial>
+  </xacro:macro>
   <xacro:macro name="scrobot_sensors">
-    <!-- RGB-D camera mechanical frame. -->
-    <link name="camera_link">
-      <visual>
+    <link name="camera_bottom_screw_frame">
+      <xacro:tiny_sensor_inertial/>
+      <visual name="d435i_visual">
+        <origin xyz="0 0 0" rpy="0 0 0"/>
         <geometry>
-          <box size="0.06 0.10 0.05"/>
+          <mesh filename="package://scrobot_description/meshes/visual/d435i.STL" scale="1 1 1"/>
         </geometry>
-        <material name="scrobot_sensor"/>
+        <material name="sensor_blue"/>
       </visual>
-      <inertial>
-        <origin xyz="0 0 0" rpy="0 0 0"/>
-        <mass value="0.2"/>
-        <inertia
-          ixx="0.00021"
-          ixy="0.0"
-          ixz="0.0"
-          iyy="0.00010"
-          iyz="0.0"
-          izz="0.00023"/>
-      </inertial>
     </link>
-    <joint name="camera_joint" type="fixed">
+    <joint name="camera_mount_joint" type="fixed">
       <parent link="base_link"/>
+      <child link="camera_bottom_screw_frame"/>
+      <origin
+        xyz="${camera_x} ${camera_y} ${camera_z}"
+        rpy="${camera_roll} ${camera_pitch} ${camera_yaw}"/>
+    </joint>
+    <link name="camera_link"><xacro:tiny_sensor_inertial/></link>
+    <joint name="camera_link_joint" type="fixed">
+      <parent link="camera_bottom_screw_frame"/>
       <child link="camera_link"/>
-      <!-- Placeholder mounting pose relative to base_link. -->
-      <origin xyz="0.18 0 0.23" rpy="0 0 0"/>
+      <origin xyz="0.0106 0.0175 0.0125" rpy="0 0 0"/>
     </joint>
-    <!--
-      ROS optical-frame convention:
-        +Z forward through the lens
-        +X right in the image
-        +Y down in the image
-    -->
-    <link name="camera_color_optical_frame"/>
-    <joint name="camera_color_optical_joint" type="fixed">
+    <link name="camera_depth_frame"/>
+    <joint name="camera_depth_joint" type="fixed">
       <parent link="camera_link"/>
-      <child link="camera_color_optical_frame"/>
-      <origin xyz="0 0 0" rpy="${-pi / 2.0} 0 ${-pi / 2.0}"/>
+      <child link="camera_depth_frame"/>
+      <origin xyz="0 0 0" rpy="0 0 0"/>
     </joint>
     <link name="camera_depth_optical_frame"/>
     <joint name="camera_depth_optical_joint" type="fixed">
+      <parent link="camera_depth_frame"/>
+      <child link="camera_depth_optical_frame"/>
+      <origin xyz="0 0 0" rpy="${-pi/2} 0 ${-pi/2}"/>
+    </joint>
+    <link name="camera_infra1_frame"/>
+    <joint name="camera_infra1_joint" type="fixed">
       <parent link="camera_link"/>
-      <child link="camera_depth_optical_frame"/>
-      <origin xyz="0 0 0" rpy="${-pi / 2.0} 0 ${-pi / 2.0}"/>
+      <child link="camera_infra1_frame"/>
+      <origin xyz="0 0 0" rpy="0 0 0"/>
     </joint>
-    <!-- IMU frame. Mounting pose is a placeholder. -->
-    <link name="imu_link">
-      <visual>
-        <geometry>
-          <box size="0.04 0.04 0.015"/>
-        </geometry>
-        <material name="scrobot_sensor"/>
-      </visual>
-      <inertial>
-        <origin xyz="0 0 0" rpy="0 0 0"/>
-        <mass value="0.05"/>
-        <inertia
-          ixx="0.0000076"
-          ixy="0.0"
-          ixz="0.0"
-          iyy="0.0000076"
-          iyz="0.0"
-          izz="0.0000133"/>
-      </inertial>
-    </link>
+    <link name="camera_infra1_optical_frame"/>
+    <joint name="camera_infra1_optical_joint" type="fixed">
+      <parent link="camera_infra1_frame"/>
+      <child link="camera_infra1_optical_frame"/>
+      <origin xyz="0 0 0" rpy="${-pi/2} 0 ${-pi/2}"/>
+    </joint>
+    <link name="camera_infra2_frame"/>
+    <joint name="camera_infra2_joint" type="fixed">
+      <parent link="camera_link"/>
+      <child link="camera_infra2_frame"/>
+      <origin xyz="0 -0.050 0" rpy="0 0 0"/>
+    </joint>
+    <link name="camera_infra2_optical_frame"/>
+    <joint name="camera_infra2_optical_joint" type="fixed">
+      <parent link="camera_infra2_frame"/>
+      <child link="camera_infra2_optical_frame"/>
+      <origin xyz="0 0 0" rpy="${-pi/2} 0 ${-pi/2}"/>
+    </joint>
+    <link name="camera_color_frame"/>
+    <joint name="camera_color_joint" type="fixed">
+      <parent link="camera_link"/>
+      <child link="camera_color_frame"/>
+      <origin xyz="0 0.015 0" rpy="0 0 0"/>
+    </joint>
+    <link name="camera_color_optical_frame"/>
+    <joint name="camera_color_optical_joint" type="fixed">
+      <parent link="camera_color_frame"/>
+      <child link="camera_color_optical_frame"/>
+      <origin xyz="0 0 0" rpy="${-pi/2} 0 ${-pi/2}"/>
+    </joint>
+    <link name="imu_link"><xacro:tiny_sensor_inertial/></link>
     <joint name="imu_joint" type="fixed">
       <parent link="base_link"/>
       <child link="imu_link"/>
-      <origin xyz="0 0 0.10" rpy="0 0 0"/>
+      <origin xyz="${imu_x} ${imu_y} ${imu_z}" rpy="0 0 0"/>
+    </joint>
+    <link name="mag_link"><xacro:tiny_sensor_inertial/></link>
+    <joint name="mag_joint" type="fixed">
+      <parent link="base_link"/>
+      <child link="mag_link"/>
+      <origin xyz="${mag_x} ${mag_y} ${mag_z}" rpy="0 0 0"/>
     </joint>
   </xacro:macro>

File: src/scrobot_description/urdf/wheels.xacro (robot description, xacro)
@@ -1,42 +1,42 @@
 <?xml version="1.0"?>
 <robot xmlns:xacro="http://www.ros.org/wiki/xacro">
-  <xacro:macro name="drive_wheel" params="name y_position">
+  <xacro:macro name="scrobot_drive_wheel" params="name y mesh_file">
     <link name="${name}_wheel_link">
-      <visual>
-        <!-- URDF cylinders are aligned with local Z; rotate them onto the Y axle. -->
-        <origin xyz="0 0 0" rpy="${pi / 2.0} 0 0"/>
+      <inertial>
+        <origin xyz="0 0 0" rpy="0 0 0"/>
+        <mass value="0.155"/>
+        <inertia
+          ixx="1.37e-4"
+          ixy="0"
+          ixz="0"
+          iyy="2.55e-4"
+          iyz="0"
+          izz="1.37e-4"/>
+      </inertial>
+      <visual name="${name}_wheel_visual">
+        <origin xyz="0 0 0" rpy="0 0 0"/>
         <geometry>
-          <cylinder radius="${wheel_radius}" length="${wheel_width}"/>
+          <mesh filename="package://scrobot_description/meshes/visual/${mesh_file}" scale="1 1 1"/>
         </geometry>
-        <material name="scrobot_dark"/>
+        <material name="rubber_black"/>
       </visual>
-      <collision>
-        <origin xyz="0 0 0" rpy="${pi / 2.0} 0 0"/>
+      <collision name="${name}_wheel_collision">
+        <origin xyz="0 0 0" rpy="${pi/2} 0 0"/>
         <geometry>
           <cylinder radius="${wheel_radius}" length="${wheel_width}"/>
         </geometry>
       </collision>
-      <inertial>
-        <origin xyz="0 0 0" rpy="0 0 0"/>
-        <mass value="0.5"/>
-        <inertia
-          ixx="${0.5 / 12.0 * (3.0 * wheel_radius * wheel_radius + wheel_width * wheel_width)}"
-          ixy="0.0"
-          ixz="0.0"
-          iyy="${0.5 / 2.0 * wheel_radius * wheel_radius}"
-          iyz="0.0"
-          izz="${0.5 / 12.0 * (3.0 * wheel_radius * wheel_radius + wheel_width * wheel_width)}"/>
-      </inertial>
     </link>
     <joint name="${name}_wheel_joint" type="continuous">
       <parent link="base_link"/>
       <child link="${name}_wheel_link"/>
-      <origin xyz="${wheel_x} ${y_position} ${wheel_radius - base_link_z}" rpy="0 0 0"/>
+      <origin xyz="0 ${y} 0" rpy="0 0 0"/>
       <axis xyz="0 1 0"/>
+      <dynamics damping="0.0" friction="0.0"/>
     </joint>
   </xacro:macro>
   <xacro:macro name="scrobot_wheels">
-    <xacro:drive_wheel name="left" y_position="${wheel_separation / 2.0}"/>
-    <xacro:drive_wheel name="right" y_position="${-wheel_separation / 2.0}"/>
+    <xacro:scrobot_drive_wheel name="left" y="${wheel_separation / 2.0}" mesh_file="left_wheel.STL"/>
+    <xacro:scrobot_drive_wheel name="right" y="${-wheel_separation / 2.0}" mesh_file="right_wheel.STL"/>
   </xacro:macro>
 </robot>

File: src/scrobot_simulation/urdf/scrobot_sim.urdf.xacro (robot description, xacro)
@@ -1,26 +1,19 @@
 <?xml version="1.0"?>
-<robot
-  xmlns:xacro="http://www.ros.org/wiki/xacro"
-  name="scrobot">
-  <!-- ============================================ -->
-  <!-- Generic robot description                    -->
-  <!-- ============================================ -->
+<robot xmlns:xacro="http://www.ros.org/wiki/xacro" name="scrobot">
+  <!-- Real robot geometry -->
   <xacro:include
     filename="$(find scrobot_description)/urdf/scrobot.urdf.xacro"/>
-  <!-- ============================================ -->
-  <!-- Gazebo sensors                               -->
-  <!-- ============================================ -->
+  <!-- Gazebo sensors -->
   <xacro:include
     filename="$(find scrobot_simulation)/urdf/sensors_gazebo.xacro"/>
-  <!-- ============================================ -->
-  <!-- ros2_control interfaces for Gazebo            -->
-  <!-- ============================================ -->
-  <ros2_control
-    name="GazeboSimSystem"
-    type="system">
+  <!-- Gazebo physical properties -->
+  <xacro:include
+    filename="$(find scrobot_simulation)/urdf/physics_gazebo.xacro"/>
+  <xacro:scrobot_gazebo_sensors/>
+  <xacro:scrobot_gazebo_physics/>
+  <ros2_control name="GazeboSimSystem" type="system">
     <hardware>
       <plugin>gz_ros2_control/GazeboSimSystem</plugin>
     </hardware>
-    <!-- Left drive wheel -->
     <joint name="left_wheel_joint">
       <command_interface name="velocity"/>
@@ -28,5 +21,4 @@
       <state_interface name="velocity"/>
     </joint>
-    <!-- Right drive wheel -->
     <joint name="right_wheel_joint">
       <command_interface name="velocity"/>
@@ -34,15 +26,26 @@
       <state_interface name="velocity"/>
     </joint>
+    <joint name="left_caster_swivel_joint">
+      <state_interface name="position"/>
+      <state_interface name="velocity"/>
+    </joint>
+    <joint name="left_caster_wheel_joint">
+      <state_interface name="position"/>
+      <state_interface name="velocity"/>
+    </joint>
+    <joint name="right_caster_swivel_joint">
+      <state_interface name="position"/>
+      <state_interface name="velocity"/>
+    </joint>
+    <joint name="right_caster_wheel_joint">
+      <state_interface name="position"/>
+      <state_interface name="velocity"/>
+    </joint>
   </ros2_control>
-  <!-- ============================================ -->
-  <!-- Gazebo ros2_control plugin                    -->
-  <!-- ============================================ -->
   <gazebo>
     <plugin
       filename="libgz_ros2_control-system.so"
       name="gz_ros2_control::GazeboSimROS2ControlPlugin">
-      <parameters>
-        $(find scrobot_control)/config/controllers.yaml
-      </parameters>
+      <parameters>$(find scrobot_control)/config/controllers.yaml</parameters>
     </plugin>
   </gazebo>
