Commit message: add model, mass, inertia and collision

File: src/scrobot_simulation/urdf/sensors_gazebo.xacro (robot description, xacro)
@@ -1,59 +1,45 @@
 <?xml version="1.0"?>
 <robot xmlns:xacro="http://www.ros.org/wiki/xacro">
-  <!-- ============================================ -->
-  <!-- Simulated IMU                                -->
-  <!-- ============================================ -->
-  <gazebo reference="imu_link">
-    <sensor name="imu_sensor" type="imu">
-      <always_on>true</always_on>
-      <update_rate>100.0</update_rate>
-      <visualize>false</visualize>
-      <topic>/imu/data</topic>
-    </sensor>
-  </gazebo>
-  <!-- ============================================ -->
-  <!-- RealSense D435i-like RGB-D camera            -->
-  <!-- ============================================ -->
-  <gazebo reference="camera_link">
-    <sensor
-      name="d435i_rgbd"
-      type="rgbd_camera">
-      <always_on>true</always_on>
-      <update_rate>30.0</update_rate>
-      <visualize>true</visualize>
-      <!--
-        Gazebo base topic.
-        Generates:
-          /camera/image
-          /camera/depth_image
-          /camera/camera_info
-          /camera/points
-      -->
-      <topic>/camera</topic>
-      <!-- Gazebo mechanical sensor frame -->
-      <gz_frame_id>camera_link</gz_frame_id>
-      <camera>
-        <!-- D435i RGB horizontal FOV ~= 69 deg -->
-        <horizontal_fov>1.20427718</horizontal_fov>
-        <image>
-          <width>640</width>
-          <height>360</height>
-          <format>R8G8B8</format>
-        </image>
-        <clip>
-          <near>0.30</near>
-          <far>3.0</far>
-        </clip>
-        <!--
-          Gazebo renders cameras with +X forward,
-          while ROS optical frames use +Z forward.
-          Your existing camera_color_optical_frame
-          already provides that transform.
-        -->
-        <optical_frame_id>
-          camera_color_optical_frame
-        </optical_frame_id>
-      </camera>
-    </sensor>
-  </gazebo>
+  <xacro:macro name="scrobot_gazebo_sensors">
+    <gazebo reference="imu_link">
+      <sensor name="imu_sensor" type="imu">
+        <always_on>true</always_on>
+        <update_rate>100.0</update_rate>
+        <visualize>false</visualize>
+        <topic>/imu/data</topic>
+        <gz_frame_id>imu_link</gz_frame_id>
+      </sensor>
+    </gazebo>
+    <gazebo reference="mag_link">
+      <sensor name="magnetometer_sensor" type="magnetometer">
+        <always_on>true</always_on>
+        <update_rate>50.0</update_rate>
+        <visualize>false</visualize>
+        <topic>/imu/mag</topic>
+        <gz_frame_id>mag_link</gz_frame_id>
+      </sensor>
+    </gazebo>
+    <gazebo reference="camera_link">
+      <sensor name="d435i_rgbd" type="rgbd_camera">
+        <always_on>true</always_on>
+        <update_rate>30.0</update_rate>
+        <visualize>true</visualize>
+        <topic>/camera</topic>
+        <gz_frame_id>camera_link</gz_frame_id>
+        <camera>
+          <horizontal_fov>1.20427718</horizontal_fov>
+          <image>
+            <width>640</width>
+            <height>360</height>
+            <format>R8G8B8</format>
+          </image>
+          <clip>
+            <near>0.30</near>
+            <far>3.0</far>
+          </clip>
+          <optical_frame_id>camera_color_optical_frame</optical_frame_id>
+        </camera>
+      </sensor>
+    </gazebo>
+  </xacro:macro>
 </robot>

Commit message: Make base footprint virtual and document mass ownership

File: src/scrobot_description/urdf/base.xacro (robot description, xacro)
@@ -2,11 +2,6 @@
 <robot xmlns:xacro="http://www.ros.org/wiki/xacro">
   <xacro:macro name="scrobot_base">
-    <link name="base_footprint">
-      <inertial>
-        <origin xyz="0 0 0" rpy="0 0 0"/>
-        <mass value="0.0001"/>
-        <inertia ixx="1e-8" ixy="0" ixz="0" iyy="1e-8" iyz="0" izz="1e-8"/>
-      </inertial>
-    </link>
+    <!-- Virtual ground-projected navigation frame; no physical inertia. -->
+    <link name="base_footprint"/>
     <joint name="base_footprint_joint" type="fixed">
       <parent link="base_footprint"/>
@@ -15,4 +10,10 @@
     </joint>
     <link name="base_link">
+      <!--
+        Authoritative CAD-derived assembled-body mass/inertia model.
+        Fixed accessories are not given additional physical mass elsewhere;
+        articulated wheel/caster inertias remain only where needed for joint
+        dynamics in simulation.
+      -->
       <inertial>
         <origin xyz="-0.060 0.002 0.195" rpy="0 0 0"/>

Commit message: Restore negligible inertia on Gazebo root frame

File: src/scrobot_description/urdf/base.xacro (robot description, xacro)
@@ -2,6 +2,15 @@
 <robot xmlns:xacro="http://www.ros.org/wiki/xacro">
   <xacro:macro name="scrobot_base">
-    <!-- Virtual ground-projected navigation frame; no physical inertia. -->
-    <link name="base_footprint"/>
+    <!--
+      Ground-projected navigation root. Keep a negligible inertia so Gazebo has
+      a physical canonical root link before the fixed base_link joint.
+    -->
+    <link name="base_footprint">
+      <inertial>
+        <origin xyz="0 0 0" rpy="0 0 0"/>
+        <mass value="0.0001"/>
+        <inertia ixx="1e-8" ixy="0" ixz="0" iyy="1e-8" iyz="0" izz="1e-8"/>
+      </inertial>
+    </link>
     <joint name="base_footprint_joint" type="fixed">
       <parent link="base_footprint"/>
