Commit message: add option for rs IMU

File: src/scrobot_description/urdf/sensors.xacro (robot description, xacro)
@@ -80,8 +80,64 @@
       <origin xyz="0 0 0" rpy="${-pi/2} 0 ${-pi/2}"/>
     </joint>
-    <link name="imu_link"><xacro:tiny_sensor_inertial/></link>
-    <joint name="imu_joint" type="fixed">
+    <!-- ========================================================= -->
+    <!-- RealSense D435i IMU                                       -->
+    <!-- Nominal extrinsics from official realsense2_description   -->
+    <!-- ========================================================= -->
+    <link name="camera_accel_frame"/>
+    <joint name="camera_accel_joint" type="fixed">
+      <parent link="camera_link"/>
+      <child link="camera_accel_frame"/>
+      <origin
+        xyz="-0.01174 -0.00552 0.00510"
+        rpy="0 0 0"/>
+    </joint>
+    <link name="camera_accel_optical_frame"/>
+    <joint name="camera_accel_optical_joint" type="fixed">
+      <parent link="camera_accel_frame"/>
+      <child link="camera_accel_optical_frame"/>
+      <origin
+        xyz="0 0 0"
+        rpy="${-pi/2} 0 ${-pi/2}"/>
+    </joint>
+    <link name="camera_gyro_frame"/>
+    <joint name="camera_gyro_joint" type="fixed">
+      <parent link="camera_link"/>
+      <child link="camera_gyro_frame"/>
+      <origin
+        xyz="-0.01174 -0.00552 0.00510"
+        rpy="0 0 0"/>
+    </joint>
+    <link name="camera_gyro_optical_frame"/>
+    <joint name="camera_gyro_optical_joint" type="fixed">
+      <parent link="camera_gyro_frame"/>
+      <child link="camera_gyro_optical_frame"/>
+      <origin
+        xyz="0 0 0"
+        rpy="${-pi/2} 0 ${-pi/2}"/>
+    </joint>
+    <!-- ========================================================= -->
+    <!-- Combined RealSense IMU frame                              -->
+    <!-- Used by /camera/camera/imu when unite_imu_method > 0      -->
+    <!-- ========================================================= -->
+    <link name="camera_imu_frame"/>
+    <joint name="camera_imu_joint" type="fixed">
+      <parent link="camera_link"/>
+      <child link="camera_imu_frame"/>
+      <origin
+        xyz="-0.01174 -0.00552 0.00510"
+        rpy="0 0 0"/>
+    </joint>
+    <link name="camera_imu_optical_frame"/>
+    <joint name="camera_imu_optical_joint" type="fixed">
+      <parent link="camera_imu_frame"/>
+      <child link="camera_imu_optical_frame"/>
+      <origin
+        xyz="0 0 0"
+        rpy="${-pi/2} 0 ${-pi/2}"/>
+    </joint>
+    <link name="bmi160_link"><xacro:tiny_sensor_inertial/></link>
+    <joint name="bmi160_joint" type="fixed">
       <parent link="base_link"/>
-      <child link="imu_link"/>
+      <child link="bmi160_link"/>
       <origin xyz="${imu_x} ${imu_y} ${imu_z}" rpy="0 0 0"/>
     </joint>

File: src/scrobot_simulation/urdf/sensors_gazebo.xacro (robot description, xacro)
@@ -2,5 +2,5 @@
 <robot xmlns:xacro="http://www.ros.org/wiki/xacro">
   <xacro:macro name="scrobot_gazebo_sensors">
-    <gazebo reference="imu_link">
+    <gazebo reference="camera_imu_frame">
       <sensor name="imu_sensor" type="imu">
         <always_on>true</always_on>
@@ -35,6 +35,6 @@
           </image>
           <clip>
-            <near>0.30</near>
-            <far>3.0</far>
+            <near>0.1</near>
+            <far>10</far>
           </clip>
           <optical_frame_id>camera_color_optical_frame</optical_frame_id>

Commit message: better global local, fixed apriltag frame

File: src/scrobot_description/urdf/sensors.xacro (robot description, xacro)
@@ -44,5 +44,5 @@
       <origin xyz="0 0 0" rpy="${-pi/2} 0 ${-pi/2}"/>
     </joint>
-    <link name="camera_infra1_frame"/>
+    <!-- <link name="camera_infra1_frame"/>
     <joint name="camera_infra1_joint" type="fixed">
       <parent link="camera_link"/>
@@ -67,5 +67,5 @@
       <child link="camera_infra2_optical_frame"/>
       <origin xyz="0 0 0" rpy="${-pi/2} 0 ${-pi/2}"/>
-    </joint>
+    </joint> -->
     <link name="camera_color_frame"/>
     <joint name="camera_color_joint" type="fixed">

File: src/scrobot_simulation/urdf/sensors_gazebo.xacro (robot description, xacro)
@@ -25,4 +25,5 @@
     <gazebo reference="camera_link">
       <sensor name="d435i_color" type="camera">
+        <pose>0 0.015 0 0 0 0</pose>
         <always_on>true</always_on>
         <update_rate>30.0</update_rate>
@@ -52,4 +53,5 @@
     <gazebo reference="camera_link">
       <sensor name="d435i_depth" type="depth_camera">
+        <pose>0 0 0 0 0 0</pose>
         <always_on>true</always_on>
         <update_rate>30.0</update_rate>

Commit message: update global_local for multitags, 1920x1080@30fps, 100mm tags

File: src/scrobot_description/urdf/sensors.xacro (robot description, xacro)
@@ -84,5 +84,5 @@
     <!-- Nominal extrinsics from official realsense2_description   -->
     <!-- ========================================================= -->
-    <link name="camera_accel_frame"/>
+    <!-- <link name="camera_accel_frame"/>
     <joint name="camera_accel_joint" type="fixed">
       <parent link="camera_link"/>
@@ -115,5 +115,5 @@
         xyz="0 0 0"
         rpy="${-pi/2} 0 ${-pi/2}"/>
-    </joint>
+    </joint> -->
     <!-- ========================================================= -->
     <!-- Combined RealSense IMU frame                              -->

Commit message: fix the realsense frame to match with real life

File: src/scrobot_description/urdf/sensors.xacro (robot description, xacro)
@@ -1,150 +1,44 @@
 <?xml version="1.0"?>
 <robot xmlns:xacro="http://www.ros.org/wiki/xacro">
+  <xacro:include
+    filename="$(find scrobot_description)/urdf/realsense_d435i.xacro"/>
   <xacro:macro name="tiny_sensor_inertial">
     <inertial>
       <origin xyz="0 0 0" rpy="0 0 0"/>
       <mass value="0.0001"/>
-      <inertia ixx="1e-8" ixy="0" ixz="0" iyy="1e-8" iyz="0" izz="1e-8"/>
+      <inertia
+        ixx="1e-8" ixy="0" ixz="0"
+        iyy="1e-8" iyz="0"
+        izz="1e-8"/>
     </inertial>
   </xacro:macro>
+  <!--
+    Robot-side sensor mounting.
+    D435i internal geometry is defined in realsense_d435i.xacro.
+    The 5883L magnetometer is a physically separate robot sensor,
+    so it remains directly attached to base_link using the existing
+    mag_x / mag_y / mag_z parameters.
+  -->
   <xacro:macro name="scrobot_sensors">
-    <link name="camera_bottom_screw_frame">
-      <xacro:tiny_sensor_inertial/>
-      <visual name="d435i_visual">
-        <origin xyz="0 0 0" rpy="0 0 0"/>
-        <geometry>
-          <mesh filename="package://scrobot_description/meshes/visual/d435i.STL" scale="1 1 1"/>
-        </geometry>
-        <material name="sensor_blue"/>
-      </visual>
-    </link>
-    <joint name="camera_mount_joint" type="fixed">
-      <parent link="base_link"/>
-      <child link="camera_bottom_screw_frame"/>
+    <!-- ====================================================== -->
+    <!-- Intel RealSense D435i                                  -->
+    <!-- ====================================================== -->
+    <xacro:scrobot_d435i parent="base_link" name="camera">
       <origin
         xyz="${camera_x} ${camera_y} ${camera_z}"
         rpy="${camera_roll} ${camera_pitch} ${camera_yaw}"/>
-    </joint>
-    <link name="camera_link"><xacro:tiny_sensor_inertial/></link>
-    <joint name="camera_link_joint" type="fixed">
-      <parent link="camera_bottom_screw_frame"/>
-      <child link="camera_link"/>
-      <origin xyz="0.0106 0.0175 0.0125" rpy="0 0 0"/>
-    </joint>
-    <link name="camera_depth_frame"/>
-    <joint name="camera_depth_joint" type="fixed">
-      <parent link="camera_link"/>
-      <child link="camera_depth_frame"/>
-      <origin xyz="0 0 0" rpy="0 0 0"/>
-    </joint>
-    <link name="camera_depth_optical_frame"/>
-    <joint name="camera_depth_optical_joint" type="fixed">
-      <parent link="camera_depth_frame"/>
-      <child link="camera_depth_optical_frame"/>
-      <origin xyz="0 0 0" rpy="${-pi/2} 0 ${-pi/2}"/>
-    </joint>
-    <!-- <link name="camera_infra1_frame"/>
-    <joint name="camera_infra1_joint" type="fixed">
-      <parent link="camera_link"/>
-      <child link="camera_infra1_frame"/>
-      <origin xyz="0 0 0" rpy="0 0 0"/>
-    </joint>
-    <link name="camera_infra1_optical_frame"/>
-    <joint name="camera_infra1_optical_joint" type="fixed">
-      <parent link="camera_infra1_frame"/>
-      <child link="camera_infra1_optical_frame"/>
-      <origin xyz="0 0 0" rpy="${-pi/2} 0 ${-pi/2}"/>
-    </joint>
-    <link name="camera_infra2_frame"/>
-    <joint name="camera_infra2_joint" type="fixed">
-      <parent link="camera_link"/>
-      <child link="camera_infra2_frame"/>
-      <origin xyz="0 -0.050 0" rpy="0 0 0"/>
-    </joint>
-    <link name="camera_infra2_optical_frame"/>
-    <joint name="camera_infra2_optical_joint" type="fixed">
-      <parent link="camera_infra2_frame"/>
-      <child link="camera_infra2_optical_frame"/>
-      <origin xyz="0 0 0" rpy="${-pi/2} 0 ${-pi/2}"/>
-    </joint> -->
-    <link name="camera_color_frame"/>
-    <joint name="camera_color_joint" type="fixed">
-      <parent link="camera_link"/>
-      <child link="camera_color_frame"/>
-      <origin xyz="0 0.015 0" rpy="0 0 0"/>
-    </joint>
-    <link name="camera_color_optical_frame"/>
-    <joint name="camera_color_optical_joint" type="fixed">
-      <parent link="camera_color_frame"/>
-      <child link="camera_color_optical_frame"/>
-      <origin xyz="0 0 0" rpy="${-pi/2} 0 ${-pi/2}"/>
-    </joint>
-    <!-- ========================================================= -->
-    <!-- RealSense D435i IMU                                       -->
-    <!-- Nominal extrinsics from official realsense2_description   -->
-    <!-- ========================================================= -->
-    <!-- <link name="camera_accel_frame"/>
-    <joint name="camera_accel_joint" type="fixed">
-      <parent link="camera_link"/>
-      <child link="camera_accel_frame"/>
-      <origin
-        xyz="-0.01174 -0.00552 0.00510"
-        rpy="0 0 0"/>
-    </joint>
-    <link name="camera_accel_optical_frame"/>
-    <joint name="camera_accel_optical_joint" type="fixed">
-      <parent link="camera_accel_frame"/>
-      <child link="camera_accel_optical_frame"/>
-      <origin
-        xyz="0 0 0"
-        rpy="${-pi/2} 0 ${-pi/2}"/>
-    </joint>
-    <link name="camera_gyro_frame"/>
-    <joint name="camera_gyro_joint" type="fixed">
-      <parent link="camera_link"/>
-      <child link="camera_gyro_frame"/>
-      <origin
-        xyz="-0.01174 -0.00552 0.00510"
-        rpy="0 0 0"/>
-    </joint>
-    <link name="camera_gyro_optical_frame"/>
-    <joint name="camera_gyro_optical_joint" type="fixed">
-      <parent link="camera_gyro_frame"/>
-      <child link="camera_gyro_optical_frame"/>
-      <origin
-        xyz="0 0 0"
-        rpy="${-pi/2} 0 ${-pi/2}"/>
-    </joint> -->
-    <!-- ========================================================= -->
-    <!-- Combined RealSense IMU frame                              -->
-    <!-- Used by /camera/camera/imu when unite_imu_method > 0      -->
-    <!-- ========================================================= -->
-    <link name="camera_imu_frame"/>
-    <joint name="camera_imu_joint" type="fixed">
-      <parent link="camera_link"/>
-      <child link="camera_imu_frame"/>
-      <origin
-        xyz="-0.01174 -0.00552 0.00510"
-        rpy="0 0 0"/>
-    </joint>
-    <link name="camera_imu_optical_frame"/>
-    <joint name="camera_imu_optical_joint" type="fixed">
-      <parent link="camera_imu_frame"/>
-      <child link="camera_imu_optical_frame"/>
-      <origin
-        xyz="0 0 0"
-        rpy="${-pi/2} 0 ${-pi/2}"/>
-    </joint>
-    <link name="bmi160_link"><xacro:tiny_sensor_inertial/></link>
-    <joint name="bmi160_joint" type="fixed">
-      <parent link="base_link"/>
-      <child link="bmi160_link"/>
-      <origin xyz="${imu_x} ${imu_y} ${imu_z}" rpy="0 0 0"/>
-    </joint>
-    <link name="mag_link"><xacro:tiny_sensor_inertial/></link>
+    </xacro:scrobot_d435i>
+    <!-- ====================================================== -->
+    <!-- Separate 5883L magnetometer                            -->
+    <!-- ====================================================== -->
+    <link name="mag_link">
+      <xacro:tiny_sensor_inertial/>
+    </link>
     <joint name="mag_joint" type="fixed">
       <parent link="base_link"/>
       <child link="mag_link"/>
-      <origin xyz="${mag_x} ${mag_y} ${mag_z}" rpy="0 0 0"/>
+      <origin
+        xyz="${mag_x} ${mag_y} ${mag_z}"
+        rpy="0 0 0"/>
     </joint>
   </xacro:macro>

File: src/scrobot_simulation/urdf/sensors_gazebo.xacro (robot description, xacro)
@@ -2,16 +2,31 @@
 <robot xmlns:xacro="http://www.ros.org/wiki/xacro">
   <xacro:macro name="scrobot_gazebo_sensors">
+    <!-- ====================================================== -->
+    <!-- D435i combined IMU                                     -->
+    <!-- ====================================================== -->
     <gazebo reference="camera_imu_frame">
-      <sensor name="imu_sensor" type="imu">
+      <sensor name="d435i_imu" type="imu">
         <always_on>true</always_on>
         <update_rate>100.0</update_rate>
         <visualize>false</visualize>
-        <topic>/imu/data</topic>
-        <gz_frame_id>imu_link</gz_frame_id>
+        <topic>/camera/imu</topic>
+        <gz_frame_id>camera_imu_frame</gz_frame_id>
+        <imu>
+          <!--
+            Match the real D435i behavior:
+            accel + gyro are available, but orientation is not
+            directly estimated by the camera.
+          -->
+          <orientation_enabled>false</orientation_enabled>
+        </imu>
       </sensor>
     </gazebo>
+    <!-- ====================================================== -->
+    <!-- Separate 5883L magnetometer                            -->
+    <!-- ====================================================== -->
     <gazebo reference="mag_link">
-      <sensor name="magnetometer_sensor" type="magnetometer">
+      <sensor name="magnetometer_5883l" type="magnetometer">
         <always_on>true</always_on>
+        <!-- Keep the previous project simulation rate. -->
         <update_rate>50.0</update_rate>
         <visualize>false</visualize>
@@ -20,20 +35,21 @@
       </sensor>
     </gazebo>
-    <!-- =============================== -->
-    <!-- D435i COLOR CAMERA              -->
-    <!-- =============================== -->
-    <gazebo reference="camera_link">
+    <!-- ====================================================== -->
+    <!-- D435i COLOR CAMERA                                     -->
+    <!-- ====================================================== -->
+    <gazebo reference="camera_color_frame">
       <sensor name="d435i_color" type="camera">
-        <pose>0 0.015 0 0 0 0</pose>
         <always_on>true</always_on>
         <update_rate>30.0</update_rate>
         <visualize>true</visualize>
         <topic>/camera/color</topic>
-        <gz_frame_id>camera_color_frame</gz_frame_id>
-        <camera>
-          <horizontal_fov>1.11701072</horizontal_fov>
+        <gz_frame_id>camera_color_optical_frame</gz_frame_id>
+        <camera name="d435i_color_camera">
+          <!-- D435i RGB HFOV ~= 69.4 deg -->
+          <horizontal_fov>1.2112585008840648</horizontal_fov>
+          <camera_info_topic>/camera/color/camera_info</camera_info_topic>
           <image>
-            <width>1280</width>
-            <height>720</height>
+            <width>1920</width>
+            <height>1080</height>
             <format>R8G8B8</format>
           </image>
@@ -42,34 +58,32 @@
             <far>20.0</far>
           </clip>
-          <optical_frame_id>
-            camera_color_optical_frame
-          </optical_frame_id>
+          <optical_frame_id>camera_color_optical_frame</optical_frame_id>
         </camera>
       </sensor>
     </gazebo>
-    <!-- =============================== -->
-    <!-- D435i DEPTH CAMERA              -->
-    <!-- =============================== -->
-    <gazebo reference="camera_link">
+    <!-- ====================================================== -->
+    <!-- D435i RAW DEPTH CAMERA                                 -->
+    <!-- ====================================================== -->
+    <gazebo reference="camera_depth_frame">
       <sensor name="d435i_depth" type="depth_camera">
-        <pose>0 0 0 0 0 0</pose>
         <always_on>true</always_on>
         <update_rate>30.0</update_rate>
         <visualize>true</visualize>
         <topic>/camera/depth</topic>
-        <gz_frame_id>camera_depth_frame</gz_frame_id>
-        <camera>
-          <horizontal_fov>1.11701072</horizontal_fov>
+        <gz_frame_id>camera_depth_optical_frame</gz_frame_id>
+        <camera name="d435i_depth_camera">
+          <!-- D435i depth HFOV ~= 87 deg -->
+          <horizontal_fov>1.5184364492350666</horizontal_fov>
+          <camera_info_topic>/camera/depth/camera_info</camera_info_topic>
           <image>
             <width>480</width>
             <height>360</height>
+            <format>R_FLOAT32</format>
           </image>
           <clip>
-            <near>0.3</near>
-            <far>3.0</far>
+            <near>0.20</near>
+            <far>6.0</far>
           </clip>
-          <optical_frame_id>
-            camera_depth_optical_frame
-          </optical_frame_id>
+          <optical_frame_id>camera_depth_optical_frame</optical_frame_id>
         </camera>
       </sensor>

Commit message: Remove abandoned external magnetometer frame

File: src/scrobot_description/urdf/sensors.xacro (robot description, xacro)
@@ -3,25 +3,8 @@
   <xacro:include
     filename="$(find scrobot_description)/urdf/realsense_d435i.xacro"/>
-  <xacro:macro name="tiny_sensor_inertial">
-    <inertial>
-      <origin xyz="0 0 0" rpy="0 0 0"/>
-      <mass value="0.0001"/>
-      <inertia
-        ixx="1e-8" ixy="0" ixz="0"
-        iyy="1e-8" iyz="0"
-        izz="1e-8"/>
-    </inertial>
-  </xacro:macro>
-  <!--
-    Robot-side sensor mounting.
-    D435i internal geometry is defined in realsense_d435i.xacro.
-    The 5883L magnetometer is a physically separate robot sensor,
-    so it remains directly attached to base_link using the existing
-    mag_x / mag_y / mag_z parameters.
-  -->
+  <!-- Robot-side sensor mounting. D435i internal geometry is defined in
+       realsense_d435i.xacro. The separate HMC5883L path was removed from the
+       final robot design; localization uses the D435i IMU only. -->
   <xacro:macro name="scrobot_sensors">
-    <!-- ====================================================== -->
-    <!-- Intel RealSense D435i                                  -->
-    <!-- ====================================================== -->
     <xacro:scrobot_d435i parent="base_link" name="camera">
       <origin
@@ -29,17 +12,4 @@
         rpy="${camera_roll} ${camera_pitch} ${camera_yaw}"/>
     </xacro:scrobot_d435i>
-    <!-- ====================================================== -->
-    <!-- Separate 5883L magnetometer                            -->
-    <!-- ====================================================== -->
-    <link name="mag_link">
-      <xacro:tiny_sensor_inertial/>
-    </link>
-    <joint name="mag_joint" type="fixed">
-      <parent link="base_link"/>
-      <child link="mag_link"/>
-      <origin
-        xyz="${mag_x} ${mag_y} ${mag_z}"
-        rpy="0 0 0"/>
-    </joint>
   </xacro:macro>
 </robot>

Commit message: Make magnetometer frame optional

File: src/scrobot_description/urdf/sensors.xacro (robot description, xacro)
@@ -3,4 +3,5 @@
   <xacro:include
     filename="$(find scrobot_description)/urdf/realsense_d435i.xacro"/>
+  <!-- Numerical placeholder only; fixed sensor mass is accounted in base_link. -->
   <xacro:macro name="tiny_sensor_inertial">
     <inertial>
@@ -20,5 +21,5 @@
     mag_x / mag_y / mag_z parameters.
   -->
-  <xacro:macro name="scrobot_sensors">
+  <xacro:macro name="scrobot_sensors" params="enable_magnetometer:=false">
     <!-- ====================================================== -->
     <!-- Intel RealSense D435i                                  -->
@@ -32,14 +33,16 @@
     <!-- Separate 5883L magnetometer                            -->
     <!-- ====================================================== -->
-    <link name="mag_link">
-      <xacro:tiny_sensor_inertial/>
-    </link>
-    <joint name="mag_joint" type="fixed">
-      <parent link="base_link"/>
-      <child link="mag_link"/>
-      <origin
-        xyz="${mag_x} ${mag_y} ${mag_z}"
-        rpy="0 0 0"/>
-    </joint>
+    <xacro:if value="${enable_magnetometer}">
+      <link name="mag_link">
+        <xacro:tiny_sensor_inertial/>
+      </link>
+      <joint name="mag_joint" type="fixed">
+        <parent link="base_link"/>
+        <child link="mag_link"/>
+        <origin
+          xyz="${mag_x} ${mag_y} ${mag_z}"
+          rpy="0 0 0"/>
+      </joint>
+    </xacro:if>
   </xacro:macro>
 </robot>

Commit message: Remove obsolete external magnetometer frame

File: src/scrobot_description/urdf/sensors.xacro (robot description, xacro)
@@ -3,25 +3,7 @@
   <xacro:include
     filename="$(find scrobot_description)/urdf/realsense_d435i.xacro"/>
-  <xacro:macro name="tiny_sensor_inertial">
-    <inertial>
-      <origin xyz="0 0 0" rpy="0 0 0"/>
-      <mass value="0.0001"/>
-      <inertia
-        ixx="1e-8" ixy="0" ixz="0"
-        iyy="1e-8" iyz="0"
-        izz="1e-8"/>
-    </inertial>
-  </xacro:macro>
-  <!--
-    Robot-side sensor mounting.
-    D435i internal geometry is defined in realsense_d435i.xacro.
-    The 5883L magnetometer is a physically separate robot sensor,
-    so it remains directly attached to base_link using the existing
-    mag_x / mag_y / mag_z parameters.
-  -->
   <xacro:macro name="scrobot_sensors">
-    <!-- ====================================================== -->
-    <!-- Intel RealSense D435i                                  -->
-    <!-- ====================================================== -->
+    <!-- Intel RealSense D435i. Internal camera/IMU frame geometry lives in
+         realsense_d435i.xacro; this origin is the measured robot mount. -->
     <xacro:scrobot_d435i parent="base_link" name="camera">
       <origin
@@ -29,17 +11,4 @@
         rpy="${camera_roll} ${camera_pitch} ${camera_yaw}"/>
     </xacro:scrobot_d435i>
-    <!-- ====================================================== -->
-    <!-- Separate 5883L magnetometer                            -->
-    <!-- ====================================================== -->
-    <link name="mag_link">
-      <xacro:tiny_sensor_inertial/>
-    </link>
-    <joint name="mag_joint" type="fixed">
-      <parent link="base_link"/>
-      <child link="mag_link"/>
-      <origin
-        xyz="${mag_x} ${mag_y} ${mag_z}"
-        rpy="0 0 0"/>
-    </joint>
   </xacro:macro>
 </robot>
