Commit message: tried to fix speed by splitting rgb and depth config

File: src/scrobot_description/urdf/scrobot.urdf.xacro (robot description, xacro)
@@ -36,7 +36,7 @@
   <xacro:property name="collector_y" value="0.0"/>
   <xacro:property name="collector_z" value="-0.020"/>
-  <xacro:property name="camera_x" value="0.130"/>
+  <xacro:property name="camera_x" value="0.12"/>
   <xacro:property name="camera_y" value="0.0"/>
-  <xacro:property name="camera_z" value="0.225"/>
+  <xacro:property name="camera_z" value="0.22"/>
   <xacro:property name="camera_roll" value="0.0"/>
   <xacro:property name="camera_pitch" value="${7.0 * pi / 180.0}"/>

File: src/scrobot_simulation/urdf/sensors_gazebo.xacro (robot description, xacro)
@@ -20,23 +20,54 @@
       </sensor>
     </gazebo>
+    <!-- =============================== -->
+    <!-- D435i COLOR CAMERA              -->
+    <!-- =============================== -->
     <gazebo reference="camera_link">
-      <sensor name="d435i_rgbd" type="rgbd_camera">
+      <sensor name="d435i_color" type="camera">
         <always_on>true</always_on>
         <update_rate>30.0</update_rate>
         <visualize>true</visualize>
-        <topic>/camera</topic>
-        <gz_frame_id>camera_link</gz_frame_id>
+        <topic>/camera/color</topic>
+        <gz_frame_id>camera_color_frame</gz_frame_id>
         <camera>
-          <horizontal_fov>1.20427718</horizontal_fov>
+          <horizontal_fov>1.11701072</horizontal_fov>
           <image>
-            <width>640</width>
-            <height>360</height>
+            <width>1920</width>
+            <height>1080</height>
             <format>R8G8B8</format>
           </image>
           <clip>
-            <near>0.1</near>
-            <far>10</far>
+            <near>0.05</near>
+            <far>20.0</far>
           </clip>
-          <optical_frame_id>camera_color_optical_frame</optical_frame_id>
+          <optical_frame_id>
+            camera_color_optical_frame
+          </optical_frame_id>
+        </camera>
+      </sensor>
+    </gazebo>
+    <!-- =============================== -->
+    <!-- D435i DEPTH CAMERA              -->
+    <!-- =============================== -->
+    <gazebo reference="camera_link">
+      <sensor name="d435i_depth" type="depth_camera">
+        <always_on>true</always_on>
+        <update_rate>15.0</update_rate>
+        <visualize>true</visualize>
+        <topic>/camera/depth</topic>
+        <gz_frame_id>camera_depth_frame</gz_frame_id>
+        <camera>
+          <horizontal_fov>1.11701072</horizontal_fov>
+          <image>
+            <width>1280</width>
+            <height>720</height>
+          </image>
+          <clip>
+            <near>0.3</near>
+            <far>3.0</far>
+          </clip>
+          <optical_frame_id>
+            camera_depth_frame
+          </optical_frame_id>
         </camera>
       </sensor>

Commit message: model ideal line-contact wheel width for simulation evaluation

File: src/scrobot_description/urdf/scrobot.urdf.xacro (robot description, xacro)
@@ -16,4 +16,12 @@
   <xacro:property name="wheel_width" value="0.030"/>
   <xacro:property name="wheel_separation" value="0.420"/>
+  <!--
+    Collision width can be overridden by simulation while the visual and
+    physical wheel dimensions remain 30 mm. Real/default description keeps
+    the full wheel width; Gazebo uses a narrow line-contact approximation
+    for ideal differential-drive odometry evaluation.
+  -->
+  <xacro:arg name="wheel_collision_width" default="0.030"/>
+  <xacro:property name="wheel_collision_width" value="$(arg wheel_collision_width)"/>
   <xacro:property name="base_front_x" value="0.325"/>
   <xacro:property name="base_rear_x" value="-0.450"/>
@@ -59,7 +67,4 @@
   <xacro:scrobot_sensors/>
   <!-- ====================================================== -->
-  <!-- Gazebo-only ground truth pose for evaluation           -->
-  <!-- ====================================================== -->
-  <!-- ====================================================== -->
   <!-- Gazebo-only ground truth odometry for evaluation       -->
   <!-- ====================================================== -->

Commit message: Update physical camera pitch to 15 degrees

File: src/scrobot_description/urdf/scrobot.urdf.xacro (robot description, xacro)
@@ -52,5 +52,5 @@
   <xacro:property name="camera_z" value="0.22"/>
   <xacro:property name="camera_roll" value="0.0"/>
-  <xacro:property name="camera_pitch" value="${7.0 * pi / 180.0}"/>
+  <xacro:property name="camera_pitch" value="${15.0 * pi / 180.0}"/>
   <xacro:property name="camera_yaw" value="0.0"/>
   <xacro:property name="imu_x" value="-0.035"/>

Commit message: Align D435i mount with current robot geometry

File: src/scrobot_description/urdf/scrobot.urdf.xacro (robot description, xacro)
@@ -44,16 +44,13 @@
   <xacro:property name="collector_y" value="0.0"/>
   <xacro:property name="collector_z" value="-0.020"/>
-  <xacro:property name="camera_x" value="0.12"/>
+  <!-- D435i tripod screw mount measured from base_link:
+       base_link origin is centered between the two drive wheels.
+       Positive pitch rotates the camera optical axis downward here. -->
+  <xacro:property name="camera_x" value="0.110"/>
   <xacro:property name="camera_y" value="0.0"/>
-  <xacro:property name="camera_z" value="0.22"/>
+  <xacro:property name="camera_z" value="0.2275"/>
   <xacro:property name="camera_roll" value="0.0"/>
-  <xacro:property name="camera_pitch" value="${7.0 * pi / 180.0}"/>
+  <xacro:property name="camera_pitch" value="${15.0 * pi / 180.0}"/>
   <xacro:property name="camera_yaw" value="0.0"/>
-  <xacro:property name="imu_x" value="-0.035"/>
-  <xacro:property name="imu_y" value="0.0"/>
-  <xacro:property name="imu_z" value="0.030"/>
-  <xacro:property name="mag_x" value="-0.035"/>
-  <xacro:property name="mag_y" value="0.0"/>
-  <xacro:property name="mag_z" value="0.040"/>
   <xacro:include filename="$(find scrobot_description)/urdf/base.xacro"/>
   <xacro:include filename="$(find scrobot_description)/urdf/wheels.xacro"/>

Commit message: Use measured D435i camera mount geometry

File: src/scrobot_description/urdf/scrobot.urdf.xacro (robot description, xacro)
@@ -44,9 +44,11 @@
   <xacro:property name="collector_y" value="0.0"/>
   <xacro:property name="collector_z" value="-0.020"/>
-  <xacro:property name="camera_x" value="0.12"/>
+  <!-- Measured D435i tripod-screw mount relative to base_link. -->
+  <xacro:property name="camera_x" value="0.110"/>
   <xacro:property name="camera_y" value="0.0"/>
-  <xacro:property name="camera_z" value="0.22"/>
+  <xacro:property name="camera_z" value="0.2275"/>
   <xacro:property name="camera_roll" value="0.0"/>
-  <xacro:property name="camera_pitch" value="${7.0 * pi / 180.0}"/>
+  <!-- Positive pitch points the optical axis downward in this URDF chain. -->
+  <xacro:property name="camera_pitch" value="${15.0 * pi / 180.0}"/>
   <xacro:property name="camera_yaw" value="0.0"/>
   <xacro:property name="imu_x" value="-0.035"/>

Commit message: Update final robot rear footprint dimension

File: src/scrobot_description/urdf/scrobot.urdf.xacro (robot description, xacro)
@@ -25,5 +25,5 @@
   <xacro:property name="wheel_collision_width" value="$(arg wheel_collision_width)"/>
   <xacro:property name="base_front_x" value="0.325"/>
-  <xacro:property name="base_rear_x" value="-0.450"/>
+  <xacro:property name="base_rear_x" value="-0.420"/>
   <xacro:property name="base_left_y" value="0.225"/>
   <xacro:property name="base_right_y" value="-0.225"/>

Commit message: Clean description geometry and sensor options

File: src/scrobot_description/urdf/scrobot.urdf.xacro (robot description, xacro)
@@ -1,4 +1,5 @@
 <?xml version="1.0"?>
 <robot xmlns:xacro="http://www.ros.org/wiki/xacro" name="scrobot">
+  <xacro:arg name="enable_magnetometer" default="false"/>
   <material name="aluminum_grey">
     <color rgba="0.60 0.62 0.65 1.0"/>
@@ -25,5 +26,5 @@
   <xacro:property name="wheel_collision_width" value="$(arg wheel_collision_width)"/>
   <xacro:property name="base_front_x" value="0.325"/>
-  <xacro:property name="base_rear_x" value="-0.420"/>
+  <xacro:property name="base_rear_x" value="-0.450"/>
   <xacro:property name="base_left_y" value="0.225"/>
   <xacro:property name="base_right_y" value="-0.225"/>
@@ -52,7 +53,4 @@
   <xacro:property name="camera_pitch" value="${15.0 * pi / 180.0}"/>
   <xacro:property name="camera_yaw" value="0.0"/>
-  <xacro:property name="imu_x" value="-0.035"/>
-  <xacro:property name="imu_y" value="0.0"/>
-  <xacro:property name="imu_z" value="0.030"/>
   <xacro:property name="mag_x" value="-0.035"/>
   <xacro:property name="mag_y" value="0.0"/>
@@ -67,4 +65,4 @@
   <xacro:scrobot_casters/>
   <xacro:scrobot_collector/>
-  <xacro:scrobot_sensors/>
+  <xacro:scrobot_sensors enable_magnetometer="$(arg enable_magnetometer)"/>
 </robot>

Commit message: Remove unused collector diameter property

File: src/scrobot_description/urdf/scrobot.urdf.xacro (robot description, xacro)
@@ -40,5 +40,4 @@
   <xacro:property name="caster_fork_com_z" value="-0.01513"/>
   <xacro:property name="collector_radius" value="0.030"/>
-  <xacro:property name="collector_diameter" value="0.060"/>
   <xacro:property name="collector_length" value="0.300"/>
   <xacro:property name="collector_x" value="0.165"/>

Commit message: Remove unused robot-description properties

File: src/scrobot_description/urdf/scrobot.urdf.xacro (robot description, xacro)
@@ -25,8 +25,4 @@
   <xacro:arg name="wheel_collision_width" default="0.030"/>
   <xacro:property name="wheel_collision_width" value="$(arg wheel_collision_width)"/>
-  <xacro:property name="base_front_x" value="0.325"/>
-  <xacro:property name="base_rear_x" value="-0.420"/>
-  <xacro:property name="base_left_y" value="0.225"/>
-  <xacro:property name="base_right_y" value="-0.225"/>
   <xacro:property name="caster_x" value="-0.300"/>
   <xacro:property name="caster_y" value="0.160"/>
@@ -39,7 +35,4 @@
   <xacro:property name="caster_fork_com_y" value="0.0"/>
   <xacro:property name="caster_fork_com_z" value="-0.01513"/>
-  <xacro:property name="collector_radius" value="0.030"/>
-  <xacro:property name="collector_diameter" value="0.060"/>
-  <xacro:property name="collector_length" value="0.300"/>
   <xacro:property name="collector_x" value="0.165"/>
   <xacro:property name="collector_y" value="0.0"/>
@@ -53,7 +46,4 @@
   <xacro:property name="camera_pitch" value="${15.0 * pi / 180.0}"/>
   <xacro:property name="camera_yaw" value="0.0"/>
-  <xacro:property name="imu_x" value="-0.035"/>
-  <xacro:property name="imu_y" value="0.0"/>
-  <xacro:property name="imu_z" value="0.030"/>
   <xacro:property name="mag_x" value="-0.035"/>
   <xacro:property name="mag_y" value="0.0"/>

Commit message: Add opt-in STM32 ros2_control to current robot description

File: src/scrobot_description/urdf/scrobot.urdf.xacro (robot description, xacro)
@@ -16,4 +16,9 @@
   <xacro:property name="wheel_width" value="0.030"/>
   <xacro:property name="wheel_separation" value="0.420"/>
+  <!-- Physical ros2_control is opt-in; simulation keeps the hardware-neutral
+       description and injects its own Gazebo control system. -->
+  <xacro:arg name="use_real_hardware" default="false"/>
+  <xacro:arg name="serial_port" default="/dev/ttyTHS1"/>
+  <xacro:arg name="baud_rate" default="1000000"/>
   <!--
     Collision width can be overridden by simulation while the visual and
@@ -46,7 +51,4 @@
   <xacro:property name="camera_pitch" value="${15.0 * pi / 180.0}"/>
   <xacro:property name="camera_yaw" value="0.0"/>
-  <xacro:property name="mag_x" value="-0.035"/>
-  <xacro:property name="mag_y" value="0.0"/>
-  <xacro:property name="mag_z" value="0.040"/>
   <xacro:include filename="$(find scrobot_description)/urdf/base.xacro"/>
   <xacro:include filename="$(find scrobot_description)/urdf/wheels.xacro"/>
@@ -54,4 +56,5 @@
   <xacro:include filename="$(find scrobot_description)/urdf/collector.xacro"/>
   <xacro:include filename="$(find scrobot_description)/urdf/sensors.xacro"/>
+  <xacro:include filename="$(find scrobot_description)/urdf/ros2_control_real.xacro"/>
   <xacro:scrobot_base/>
   <xacro:scrobot_wheels/>
@@ -59,3 +62,8 @@
   <xacro:scrobot_collector/>
   <xacro:scrobot_sensors/>
+  <xacro:if value="$(arg use_real_hardware)">
+    <xacro:scrobot_real_ros2_control
+      serial_port="$(arg serial_port)"
+      baud_rate="$(arg baud_rate)"/>
+  </xacro:if>
 </robot>
