Commit message: Expose Gazebo wheel friction tuning parameters

File: src/scrobot_simulation/urdf/physics_gazebo.xacro (robot description, xacro)
@@ -1,5 +1,7 @@
 <?xml version="1.0"?>
 <robot xmlns:xacro="http://www.ros.org/wiki/xacro">
-  <xacro:macro name="scrobot_gazebo_physics">
+  <xacro:macro
+    name="scrobot_gazebo_physics"
+    params="drive_contact_mu:=5.0 caster_contact_mu:=0.05">
     <!-- ============================================================ -->
     <!-- Physical-width drive-wheel contact tuned for stable traction -->
@@ -15,6 +17,6 @@
     -->
     <gazebo reference="left_wheel_link">
-      <mu1>5.0</mu1>
-      <mu2>5.0</mu2>
+      <mu1>${drive_contact_mu}</mu1>
+      <mu2>${drive_contact_mu}</mu2>
       <fdir1>1 0 0</fdir1>
       <slip1>0.0</slip1>
@@ -23,6 +25,6 @@
     </gazebo>
     <gazebo reference="right_wheel_link">
-      <mu1>5.0</mu1>
-      <mu2>5.0</mu2>
+      <mu1>${drive_contact_mu}</mu1>
+      <mu2>${drive_contact_mu}</mu2>
       <fdir1>1 0 0</fdir1>
       <slip1>0.0</slip1>
@@ -39,11 +41,11 @@
     -->
     <gazebo reference="left_caster_wheel_link">
-      <mu1>0.05</mu1>
-      <mu2>0.05</mu2>
+      <mu1>${caster_contact_mu}</mu1>
+      <mu2>${caster_contact_mu}</mu2>
       <maxContacts>10</maxContacts>
     </gazebo>
     <gazebo reference="right_caster_wheel_link">
-      <mu1>0.05</mu1>
-      <mu2>0.05</mu2>
+      <mu1>${caster_contact_mu}</mu1>
+      <mu2>${caster_contact_mu}</mu2>
       <maxContacts>10</maxContacts>
     </gazebo>
